Commit message: Parametrizar ruta de controllers para ros2_control y pulir comentarios
Agent-Logs-Url: https://github.com/Dominguito1/Proyecto-Final-Robotica/sessions/57ae22ec-99ae-4fe1-b8df-e59cb009e444

Co-authored-by: Dominguito1 <159958034+Dominguito1@users.noreply.github.com>

File: robot.urdf.xacro (robot description, xacro)
@@ -2,4 +2,5 @@
 <robot name="diff_bot" xmlns:xacro="http://www.ros.org/wiki/xacro">
   <xacro:arg name="use_ros2_control" default="false"/>
+  <xacro:arg name="controllers_file" default="controllers.yaml"/>
   <link name="base_link">
     <visual>
@@ -79,5 +80,6 @@
     <xacro:ros2_control_system
       left_wheel_joint="left_wheel_joint"
-      right_wheel_joint="right_wheel_joint"/>
+      right_wheel_joint="right_wheel_joint"
+      controllers_file="$(arg controllers_file)"/>
   </xacro:if>
   <xacro:unless value="$(arg use_ros2_control)">

File: ros2_control.xacro (robot description, xacro)
@@ -1,5 +1,5 @@
 <?xml version="1.0"?>
 <robot xmlns:xacro="http://www.ros.org/wiki/xacro">
-  <xacro:macro name="ros2_control_system" params="left_wheel_joint right_wheel_joint">
+  <xacro:macro name="ros2_control_system" params="left_wheel_joint right_wheel_joint controllers_file">
     <ros2_control name="GazeboSystem" type="system">
       <hardware>
@@ -19,5 +19,5 @@
     <gazebo>
       <plugin name="gazebo_ros2_control" filename="libgazebo_ros2_control.so">
-        <parameters>controllers.yaml</parameters>
+        <parameters>${controllers_file}</parameters>
       </plugin>
     </gazebo>
